File: Hardware/Hornet UFC 020a.brd (EAGLE design)
At the start: 180 x 140 mm, 102 parts, among them CN2 JST-PH-B4B-PH-SM4THRU-HOLE, SW1 ADF_SMALL

Commit message: Corrections for incorrect parts in BoM  and labeled on Schematic
Parts:
- #0, #1, #2, #3, #4, #5, #6, #7, #8, #9, A/P, BCN, CLR, D/L, EMCON, ENT, I/P, IFF, ILS, ODU1, ODU2, ODU3, ODU4, ODU5, ON/OFF, TCN: device 000_nl2:GATERON-LED -> Hornet UFC 020a:GATERON-LED
- 74HC138: value CD74HC238M -> CD74HC138M; device 000_nl2:SOIC127P600X175-16N -> Hornet UFC 020a:SOIC127P600X175-16N
- BRT, U$21, U$5, VOL1, VOL2: device 000_nl2:ENCODER+SWITCH_LARGER_TABS -> Hornet UFC 020a:ENCODER+SWITCH_LARGER_TABS
- CHANNEL1: device 000_nl2:PSC05-11 -> Hornet UFC 020a:PSC05-11
- D1, D2: value BAT54TW-7-F -> BAT54CDW-7-F; device 000_nl2:SSOT6 -> Hornet UFC 020a:SSOT6
- DIS1, DIS2, DIS3, ODU_DSP_1, ODU_DSP_2, ODU_DSP_3, ODU_DSP_5: device 000_nl2:HDLX2416(SOCKETED) -> Hornet UFC 020a:HDLX2416(SOCKETED)
- U$11, U$4: device 000_nl2:ENCODER_RGB -> Hornet UFC 020a:ENCODER_RGB
- U$31: device 000_nl2:SOIC28 -> Hornet UFC 020a:SOIC28
- U$37: value OLED_128X32_I2C_DISPLAYMODULE -> OLED_128X32_I2C_DISPLAYTHROUGH_HOLE; device 000_nl2:OLED128X32_GRAPHICS_MODULE -> Hornet UFC 020a:OLED128X32_GRAPHICS_MODULE
- U$7: value PCF8575CTSSOP24 -> PCF8575PWR; device 000_nl2:TSSOP24 -> Hornet UFC 020a:TSSOP24
