File: Hardware/Hornet UFC 020a.sch (EAGLE design)
At the start: 97 parts, among them CN2 JST-PH-B4B-PH-SM4THRU-HOLE, SW1 ADF_SMALL

Commit message: Corrections for incorrect parts in BoM  and labeled on Schematic
Parts:
- #0, #1, #2, #3, #4, #5, #6, #7, #8, #9, A/P, BCN, CLR, D/L, EMCON, ENT, I/P, IFF, ILS, ODU1, ODU2, ODU3, ODU4, ODU5, ON/OFF, TCN: device 000_nl2:GATERON-LED -> Hornet UFC 020a:GATERON-LED
- 74HC138: value CD74HC238M -> CD74HC138M; device 000_nl2:CD74HC238M -> Hornet UFC 020a:CD74HC138M
- BRT, U$21, U$5, VOL1, VOL2: device 000_nl2:ALPS_ENCODER+PUSHSWITCHLARGE_TABS -> Hornet UFC 020a:ALPS_ENCODER+PUSHSWITCHLARGE_TABS
- CHANNEL1: device 000_nl2:16-SEG_THROUGH_HOLEPSC05-11 -> Hornet UFC 020a:16-SEG_THROUGH_HOLEPSC05-11
- D1, D2: value BAT54TW-7-F -> BAT54CDW-7-F; device 000_nl2:BAT54TW-7-F -> Hornet UFC 020a:BAT54CDW-7-F
- DIS1, DIS2, DIS3, ODU_DSP_1, ODU_DSP_2, ODU_DSP_3, ODU_DSP_5: device 000_nl2:HDLX2416SOCKETED -> Hornet UFC 020a:HDLX2416SOCKETED
- U$11, U$4: device 000_nl2:ENCODER_RGB_SWITCHTHROUGHHOLE -> Hornet UFC 020a:ENCODER_RGB_SWITCHTHROUGHHOLE
- U$31: device 000_nl2:HOLTEK_HT16K33 -> Hornet UFC 020a:HOLTEK_HT16K33
- U$37: value OLED_128X32_I2C_DISPLAYMODULE -> OLED_128X32_I2C_DISPLAYTHROUGH_HOLE; device 000_nl2:OLED_128X32_I2C_DISPLAYMODULE -> Hornet UFC 020a:OLED_128X32_I2C_DISPLAYTHROUGH_HOLE
- U$7: value PCF8575CTSSOP24 -> PCF8575PWR; device 000_nl2:PCF8575CTSSOP24 -> Hornet UFC 020a:PCF8575PWR
Connections:
- net N$11: now also 74HC138.~Y7; no longer 74HC138.(~Y7)_Y7
- net N$13: now also 74HC138.~Y6; no longer 74HC138.Y6_(~Y6)
- net N$14: now also 74HC138.~Y4; no longer 74HC138.Y4_(~Y4)
- net N$15: now also 74HC138.~Y3; no longer 74HC138.Y3_(~Y3)
- net N$16: now also 74HC138.~Y2; no longer 74HC138.Y2_(~Y2)
- net N$17: now also 74HC138.~Y1; no longer 74HC138.Y1_(~Y1)
- net N$18: now also 74HC138.~Y0; no longer 74HC138.Y0_(~Y0)
- net N$9: now also 74HC138.~Y5; no longer 74HC138.Y5_(~Y5)
Other:
- note added: "Issues Identified after Manufacture ------------------------------------------- 1) NodeLua board width is 5.08 mm too much 2) DONE - LEDs D3 is incorrectly linked to Row 0 instead of 9. 3) DONE - Chip enable lines need to be inverted. This should be done by replacing the 74HC238 with a 74HC138. 4) PCF8575 is a TSSOP24 package"
- note removed: "Issues Identified after Manufacture ------------------------------------------- 1) NodeLua board width is 5.08 mm too much 2) DONE - LEDs D3 is incorrectly linked to Row 0 instead of 9. 3) DONE - Chip enable lines need to be inverted. This should be done by replacing the 74HC238 with a 74HC138."
